File: schematic/_autosave-IotDuckCoopRaspberryShield.kicad_sch (KiCad schematic)
At the start: 3 parts

Commit message: some work
Parts:
- added U1: ~, symbol raspberry:light_
Other:
- note added: "Power source"
